File: pcb/pcb.kicad_pcb (KiCad board)
At the start: 2 copper layers, 186 parts, among them J1 USB_mini_micro_B, K1 KEYSW, K10 KEYSW, K11 KEYSW, K12 KEYSW, K13 KEYSW, K14 KEYSW, K15 KEYSW, K16 KEYSW, K17 KEYSW, K18 KEYSW, K19 KEYSW, K2 KEYSW, K20 KEYSW, K21 KEYSW, K22 KEYSW, K23 KEYSW, K24 KEYSW, K25 KEYSW, K26 KEYSW, K27 KEYSW, K28 KEYSW, K29 KEYSW, K3 KEYSW, K30 KEYSW, K31 KEYSW, K32 KEYSW, K33 KEYSW, K34 KEYSW, K35 KEYSW, K36 KEYSW, K37 KEYSW, K38 KEYSW, K39 KEYSW, K4 KEYSW, K40 KEYSW, K41 KEYSW, K42 KEYSW, K43 KEYSW, K44 KEYSW, K45 KEYSW, K46 KEYSW, K47 KEYSW, K48 KEYSW, K49 KEYSW, K5 KEYSW, K50 KEYSW, K51 KEYSW, K52 KEYSW, K53 KEYSW, K54 KEYSW, K55 KEYSW, K56 KEYSW, K57 KEYSW, K58 KEYSW, K59 KEYSW, K6 KEYSW, K60 KEYSW, K61 KEYSW, K62 KEYSW, K63 KEYSW, K64 KEYSW, K65 KEYSW, K66 KEYSW, K67 KEYSW, K68 KEYSW, K69 KEYSW, K7 KEYSW, K70 KEYSW, K71 KEYSW, K72 KEYSW, K73 KEYSW, K74 KEYSW, K75 KEYSW, K76 KEYSW, K77 KEYSW, K78 KEYSW, K79 KEYSW, K8 KEYSW, K80 KEYSW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

Commit message: Updated PCB
added tracks for all the switches (whew!)
Parts:
- moved R3 8.98 mm to (174.0, 118.1)
- moved SW1 8.98 mm to (181.6, 118.1)
- moved R1 5.48 mm to (245.5, 25.0), turned to 270 degrees
- moved R2 5.39 mm to (241.0, 25.0), turned to 270 degrees
- moved C3 5.08 mm to (217.8, 132.7)
- moved C4 5.08 mm to (217.8, 122.6)
- moved R4 5.08 mm to (217.8, 127.6)
- moved C7 2.54 mm to (198.1, 114.3)
- moved C8 1.27 mm to (209.6, 114.3)
- moved D62 1.27 mm to (214.6, 83.8)
- moved U1 1.27 mm to (203.8, 127.6)
- moved C1 1.27 mm to (193.0, 114.3), turned to 90 degrees
- moved C2 1.27 mm to (189.9, 122.6)
- moved C5 1.27 mm to (189.9, 132.7)
- moved C6 1.27 mm to (189.9, 127.6)
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Routing:
- net /row0: track 0.00 -> 340.8 mm
- net /row1: track 0.00 -> 340.5 mm
- net /row2: track 0.00 -> 340.4 mm
- net /row4: track 0.00 -> 339.5 mm
- net /row3: track 0.00 -> 339.2 mm
- net Net-(K13-Pad1): track 0.00 -> 84.9 mm
- net Net-(K17-Pad1): track 0.00 -> 84.4 mm
- net Net-(K10-Pad1): track 0.00 -> 84.2 mm
- net Net-(K16-Pad1): track 0.00 -> 84.2 mm
- net Net-(K23-Pad1): track 0.00 -> 84.2 mm
- net Net-(K11-Pad1): track 0.00 -> 84.2 mm
- net Net-(K24-Pad1): track 0.00 -> 84.2 mm
- net Net-(K12-Pad1): track 0.00 -> 84.2 mm
- net Net-(K25-Pad1): track 0.00 -> 84.1 mm
- net Net-(K21-Pad1): track 0.00 -> 84.1 mm
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- added copper zone on B.Cu, net GND
- added copper zone on F.Cu, net GND
Other:
- board outline added: 325.1 x 124.5 mm

Commit message: Updated PCB
pcb is unfinished and will need serious tuneups to get it off the ground, if I ever do so
Routing:
- net Net-(R1-Pad2): track 0.00 -> 5.39 mm, vias 0 -> 1
- net Net-(R2-Pad2): track 0.00 -> 5.18 mm, vias 0 -> 1
- net /row4: track 339.5 -> 340.8 mm
